File: pcb/mixed_signal_controller.kicad_pcb (KiCad board)
At the start: 2 copper layers, 118.1 x 54.6 mm, 64 parts, among them P1 PWR_JACK_2.5x5.5, P2 HEADER_01X03, P3 BNC_DOUBLE_RA, P4 HEADER_02X08_SMD, P5 HEADER_02X08_SMD, P6 HEADER_02X08_SMD, P7 HEADER_02X08_SMD, SW1 SPST_SERIES_M, SW2 KT_SWITCH, U1 MAX6817, U2 MAX6817, U3 TLE723X, U4 TLE723X, U5 TLE723X, U6 TLE723X

Commit message: Finished pcb v1.0.
Parts:
- removed C6, C7, C8, C9: 0.1uF, mixed_signal_controller:SM1210
- removed D10, D11, D12, D13, D14, D15, D16, D17, D18, D19, D2, D20, D21, D22, D23, D24, D25, D26, D27, D28, D29, D3, D30, D31, D32, D33, D4, D5, D6, D7, D8, D9: LED_24V, mixed_signal_controller:LED_555-3XXX
- removed P5, P6, P7: HEADER_02X08_SMD, mixed_signal_controller:HEADER_02x08_SMD
- removed U3, U4, U5, U6: TLE723X, mixed_signal_controller:TLE723X
- P4: value HEADER_02X08_SMD -> HEADER_02X05_SMD; footprint mixed_signal_controller:HEADER_02x08_SMD -> mixed_signal_controller:HEADER_02x05_SMD
- moved P4 14.2 mm to (157.5, 102.9)
Connections:
- ARDUINO1 pad 48: /IN -> /BNC_A
- ARDUINO1 pad 49: /CS -> Net-(ARDUINO1-Pad49)
- ARDUINO1 pad 50: /MISO -> Net-(ARDUINO1-Pad50)
- ARDUINO1 pad 51: /MOSI -> Net-(ARDUINO1-Pad51)
- ARDUINO1 pad 52: /SCK -> Net-(ARDUINO1-Pad52)
- ARDUINO1 pad A0: /BNC_A -> /A0
- ARDUINO1 pad A1: Net-(ARDUINO1-PadA1) -> /A1
- ARDUINO1 pad A2: Net-(ARDUINO1-PadA2) -> /A2
- ARDUINO1 pad A3: Net-(ARDUINO1-PadA3) -> /A3
- ARDUINO1 pad A4: Net-(ARDUINO1-PadA4) -> /A4
- ARDUINO1 pad A5: Net-(ARDUINO1-PadA5) -> /A5
- ARDUINO1 pad A6: Net-(ARDUINO1-PadA6) -> /A6
- ARDUINO1 pad A7: Net-(ARDUINO1-PadA7) -> /A7
- ARDUINO1 pad RST: /RST -> Net-(ARDUINO1-PadRST)
- P4 pad 1: VAA -> +5V
- P4 pad 10: /OUT4 -> /A7
- P4 pad 2: /OUT0 -> GND
- P4 pad 3: VAA -> /A0
- P4 pad 4: /OUT1 -> /A1
- P4 pad 5: VAA -> /A2
- P4 pad 6: /OUT2 -> /A3
- P4 pad 7: VAA -> /A4
- P4 pad 8: /OUT3 -> /A5
- P4 pad 9: VAA -> /A6
Routing:
- net /CS: track 171.1 -> 0.00 mm, vias 3 -> 0
- net /RST: track 164.0 -> 0.00 mm, vias 3 -> 0
- net /SCK: track 153.6 -> 0.00 mm, vias 4 -> 0
- net GND: track 445.6 -> 295.8 mm, vias 6 -> 2
- net /IN: track 141.0 -> 0.00 mm, vias 5 -> 0
- net /LED_PWR: track 184.2 -> 45.6 mm, vias 3 -> 0
- net +5V: track 260.3 -> 122.4 mm, vias 1 -> 2
- net VAA: track 203.1 -> 67.5 mm, vias 1 -> 0
- net /MISO: track 77.6 -> 0.00 mm, vias 2 -> 0
- net /MOSI: track 65.0 -> 0.00 mm, vias 1 -> 0
- net /A1: track 0.00 -> 51.5 mm
- net /A3: track 0.00 -> 47.8 mm
- net /SI1: track 47.6 -> 0.00 mm
- net /A0: track 0.00 -> 47.0 mm
- net /OUT16: track 43.6 -> 0.00 mm
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- added copper zone on B.Cu, net +5V
- added copper zone on F.Cu, net GND
- removed copper zone on B.Cu, net GND
- removed copper zone on F.Cu, net VAA
Other:
- board text added: "+5VDC"
- board text added: "A0"
- board text added: "A1"
- board text added: "A2"
- board text added: "A3"
- board text added: "A4"
- board text added: "A5"
- board text added: "A6"
- board text added: "A7"
- board text added: "GND"
- board text added: "Janelia Modular Device mixed_signal_controller model_number: 1120 05/2015 version 1.0"
- board text removed: "-"
- board text removed: "0"
- board text removed: "1"
- board text removed: "10"
- board text removed: "11"
- board text removed: "12"
- board text removed: "13"
- board text removed: "14"
- board text removed: "15"
- board text removed: "16"
- board text removed: "17"
- board text removed: "18"
- board text removed: "19"
- board text removed: "2"
- board text removed: "20"
- board text removed: "21"
- board text removed: "22"
- board text removed: "23"
- board text removed: "24"
- board text removed: "25"
- board text removed: "26"
- board text removed: "27"
- board text removed: "28"
- board text removed: "29"
- board text removed: "3"
- board text removed: "30"
- board text removed: "31"
- board text removed: "4"
- board text removed: "5"
- board text removed: "6"
- board text removed: "7"
- board text removed: "8"
- board text removed: "9"
- board text removed: "Janelia Modular Device mixed_signal_controller model_number: 1110 02/2015 version 1.2"

Commit message: Finished pcb v1.1.
Parts:
- removed REG1: CONV_DC_DC_12V_1A, mixed_signal_controller:DC_DC_CONV_R78C
- added P5: HEADER_02X05_SMD, mixed_signal_controller:HEADER_02x05_SMD, F.Cu at (127.0, 116.8)
- added P6: HEADER_02X07_SMD, mixed_signal_controller:HEADER_02x07_SMD, F.Cu at (127.0, 88.9)
- added P7: HEADER_02X07_SMD, mixed_signal_controller:HEADER_02x07_SMD, F.Cu at (158.8, 88.9)
- added P8: HEADER_02X07_SMD, mixed_signal_controller:HEADER_02x07_SMD, F.Cu at (158.8, 102.9)
- added P9: HEADER_02X07_SMD, mixed_signal_controller:HEADER_02x07_SMD, F.Cu at (158.8, 116.8)
- P1: value PWR_JACK_2.5x5.5 -> PWR_JACK_2.1x5.5
- moved P4 30.5 mm to (127.0, 102.9)
Connections:
- ARDUINO1 pad 10: Net-(ARDUINO1-Pad10) -> /IO4
- ARDUINO1 pad 11: Net-(ARDUINO1-Pad11) -> /IO5
- ARDUINO1 pad 12: Net-(ARDUINO1-Pad12) -> /IO6
- ARDUINO1 pad 13: Net-(ARDUINO1-Pad13) -> /IO7
- ARDUINO1 pad 22: Net-(ARDUINO1-Pad22) -> /IO8
- ARDUINO1 pad 23: Net-(ARDUINO1-Pad23) -> /IO9
- ARDUINO1 pad 24: Net-(ARDUINO1-Pad24) -> /IO10
- ARDUINO1 pad 25: Net-(ARDUINO1-Pad25) -> /IO11
- ARDUINO1 pad 26: Net-(ARDUINO1-Pad26) -> /IO12
- ARDUINO1 pad 27: Net-(ARDUINO1-Pad27) -> /IO13
- ARDUINO1 pad 28: Net-(ARDUINO1-Pad28) -> /IO14
- ARDUINO1 pad 29: Net-(ARDUINO1-Pad29) -> /IO15
- ARDUINO1 pad 30: Net-(ARDUINO1-Pad30) -> /IO16
- ARDUINO1 pad 31: Net-(ARDUINO1-Pad31) -> /IO17
- ARDUINO1 pad 32: Net-(ARDUINO1-Pad32) -> /IO18
- ARDUINO1 pad 33: Net-(ARDUINO1-Pad33) -> /IO19
- ARDUINO1 pad 34: Net-(ARDUINO1-Pad34) -> /IO20
- ARDUINO1 pad 35: Net-(ARDUINO1-Pad35) -> /IO21
- ARDUINO1 pad 36: Net-(ARDUINO1-Pad36) -> /IO22
- ARDUINO1 pad 37: Net-(ARDUINO1-Pad37) -> /IO23
- ARDUINO1 pad 38: Net-(ARDUINO1-Pad38) -> /IO31
- ARDUINO1 pad 39: Net-(ARDUINO1-Pad39) -> /IO30
- ARDUINO1 pad 40: Net-(ARDUINO1-Pad40) -> /IO29
- ARDUINO1 pad 41: Net-(ARDUINO1-Pad41) -> /IO28
- ARDUINO1 pad 42: Net-(ARDUINO1-Pad42) -> /IO27
- ARDUINO1 pad 43: Net-(ARDUINO1-Pad43) -> /IO26
- ARDUINO1 pad 44: Net-(ARDUINO1-Pad44) -> /IO25
- ARDUINO1 pad 45: Net-(ARDUINO1-Pad45) -> /IO24
- ARDUINO1 pad 6: Net-(ARDUINO1-Pad6) -> /IO0
- ARDUINO1 pad 7: Net-(ARDUINO1-Pad7) -> /IO1
- ARDUINO1 pad 8: Net-(ARDUINO1-Pad8) -> /IO2
- ARDUINO1 pad 9: Net-(ARDUINO1-Pad9) -> /IO3
- ARDUINO1 pad A10: Net-(ARDUINO1-PadA10) -> /A10
- ARDUINO1 pad A11: Net-(ARDUINO1-PadA11) -> /A11
- ARDUINO1 pad A12: Net-(ARDUINO1-PadA12) -> /A12
- ARDUINO1 pad A13: Net-(ARDUINO1-PadA13) -> /A13
- ARDUINO1 pad A14: Net-(ARDUINO1-PadA14) -> /A14
- ARDUINO1 pad A15: Net-(ARDUINO1-PadA15) -> /A15
- ARDUINO1 pad A8: Net-(ARDUINO1-PadA8) -> /A8
- ARDUINO1 pad A9: Net-(ARDUINO1-PadA9) -> /A9
- ARDUINO1 pad V_IN: /V_IN -> VAA
- C2 pad 1: /V_IN -> VAA
Routing:
- net VAA: track 67.5 -> 203.2 mm, vias 0 -> 4
- net /IO31: track 0.00 -> 109.9 mm
- net /A13: track 0.00 -> 86.6 mm, vias 0 -> 1
- net /A14: track 0.00 -> 83.9 mm, vias 0 -> 1
- net /A12: track 0.00 -> 77.2 mm, vias 0 -> 1
- net GND: track 295.8 -> 371.9 mm, vias 2 -> 5
- net /A15: track 0.00 -> 75.1 mm, vias 0 -> 1
- net /IO15: track 0.00 -> 74.3 mm
- net /V_IN: track 68.3 -> 0.00 mm
- net +5V: track 122.4 -> 189.4 mm, vias 2 -> 3
- net /A11: track 0.00 -> 61.4 mm
- net /A10: track 0.00 -> 57.7 mm, vias 0 -> 1
- net /IO11: track 0.00 -> 55.1 mm
- net /IO27: track 0.00 -> 54.9 mm, vias 0 -> 2
- net /IO30: track 0.00 -> 52.0 mm, vias 0 -> 3
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- added copper zone on B.Cu, net VAA
- removed copper zone on B.Cu, net +5V
Other:
- board text added: "+12VDC"
- board text added: "+5V"
- board text added: "0"
- board text added: "1"
- board text added: "10"
- board text added: "11"
- board text added: "12"
- board text added: "13"
- board text added: "14"
- board text added: "15"
- board text added: "16"
- board text added: "17"
- board text added: "18"
- board text added: "19"
- board text added: "2"
- board text added: "20"
- board text added: "21"
- board text added: "22"
- board text added: "23"
- board text added: "24"
- board text added: "25"
- board text added: "26"
- board text added: "27"
- board text added: "28"
- board text added: "29"
- board text added: "3"
- board text added: "30"
- board text added: "31"
- board text added: "4"
- board text added: "5"
- board text added: "6"
- board text added: "7"
- board text added: "8"
- board text added: "9"
- board text added: "A10"
- board text added: "A11"
- board text added: "A12"
- board text added: "A13"
- board text added: "A14"
- board text added: "A15"
- board text added: "A8"
- board text added: "A9"
- board text added: "Janelia Modular Device mixed_signal_controller model_number: 1120 05/2015 version 1.1"
- board text added: "VAA"
- board text removed: "+24VDC"
- board text removed: "+5VDC"
- board text removed: "Janelia Modular Device mixed_signal_controller model_number: 1120 05/2015 version 1.0"

Commit message: JaneliaSciComp -> janelia-modular-devices.
Other:
- board text added: "https://github.com/janelia-modular-devices/modular-devices"
- board text removed: "https://github.com/JaneliaSciComp/modular-devices"
Changed lines of the file:
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@@
     (effects (font (size 1.016 1.016) (thickness 0.254)))
   )
-  (gr_text https://github.com/JaneliaSciComp/modular-devices (at 189.23 102.87 90) (layer F.SilkS)
+  (gr_text https://github.com/janelia-modular-devices/modular-devices (at 189.23 102.87 90) (layer F.SilkS)
     (effects (font (size 0.762 0.762) (thickness 0.1905)))
   )

Commit message: SPST switch -> DPST switch.
Parts:
- removed R3: 5.11k, mixed_signal_controller:SM1210
- SW1: value SPST_SERIES_M -> DPST_SERIES_M; footprint mixed_signal_controller:SPST_SERIES_M -> mixed_signal_controller:DPST_SERIES_M
- moved C2 31.1 mm to (204.5, 85.7), turned to 0 degrees
- moved P4 14.0 mm to (127.0, 116.8)
- moved P5 14.0 mm to (127.0, 102.9)
- moved D1 9.69 mm to (182.2, 111.1), turned to 270 degrees
- moved SW1 0.63 mm to (182.2, 102.9)
Connections:
- net /D_LED_PWR renamed /D_LIGHTS
- ARDUINO1 pad 10: /IO4 -> Net-(ARDUINO1-Pad10)
- ARDUINO1 pad 11: /IO5 -> Net-(ARDUINO1-Pad11)
- ARDUINO1 pad 12: /IO6 -> /BNC_A
- ARDUINO1 pad 13: /IO7 -> Net-(ARDUINO1-Pad13)
- ARDUINO1 pad 22: /IO8 -> /IO7
- ARDUINO1 pad 23: /IO9 -> /IO6
- ARDUINO1 pad 24: /IO10 -> /IO5
- ARDUINO1 pad 25: /IO11 -> /IO4
- ARDUINO1 pad 26: /IO12 -> /IO3
- ARDUINO1 pad 27: /IO13 -> /IO2
- ARDUINO1 pad 28: /IO14 -> /IO1
- ARDUINO1 pad 29: /IO15 -> /IO0
- ARDUINO1 pad 30: /IO16 -> /IO15
- ARDUINO1 pad 31: /IO17 -> /IO14
- ARDUINO1 pad 32: /IO18 -> /IO13
- ARDUINO1 pad 33: /IO19 -> /IO12
- ARDUINO1 pad 34: /IO20 -> /IO11
- ARDUINO1 pad 35: /IO21 -> /IO10
- ARDUINO1 pad 36: /IO22 -> /IO9
- ARDUINO1 pad 37: /IO23 -> /IO8
- ARDUINO1 pad 38: /IO31 -> /IO23
- ARDUINO1 pad 39: /IO30 -> /IO22
- ARDUINO1 pad 40: /IO29 -> /IO21
- ARDUINO1 pad 41: /IO28 -> /IO20
- ARDUINO1 pad 42: /IO27 -> /IO19
- ARDUINO1 pad 43: /IO26 -> /IO18
- ARDUINO1 pad 44: /IO25 -> /IO17
- ARDUINO1 pad 45: /IO24 -> /IO16
- ARDUINO1 pad 46: Net-(ARDUINO1-Pad46) -> /IO31
- ARDUINO1 pad 47: Net-(ARDUINO1-Pad47) -> /IO30
- ARDUINO1 pad 48: /BNC_A -> /IO29
- ARDUINO1 pad 49: Net-(ARDUINO1-Pad49) -> /IO28
- ARDUINO1 pad 50: Net-(ARDUINO1-Pad50) -> /IO27
- ARDUINO1 pad 51: Net-(ARDUINO1-Pad51) -> /IO26
- ARDUINO1 pad 52: Net-(ARDUINO1-Pad52) -> /IO25
- ARDUINO1 pad 53: Net-(ARDUINO1-Pad53) -> /IO24
- ARDUINO1 pad 6: /IO0 -> Net-(ARDUINO1-Pad6)
- ARDUINO1 pad 7: /IO1 -> Net-(ARDUINO1-Pad7)
- ARDUINO1 pad 8: /IO2 -> Net-(ARDUINO1-Pad8)
- ARDUINO1 pad 9: /IO3 -> Net-(ARDUINO1-Pad9)
- ARDUINO1 pad A0: /A0 -> /A7
- ARDUINO1 pad A1: /A1 -> /A5
- ARDUINO1 pad A10: /A10 -> /A11
- ARDUINO1 pad A11: /A11 -> /A9
- ARDUINO1 pad A12: /A12 -> /A14
- ARDUINO1 pad A13: /A13 -> /A12
- ARDUINO1 pad A14: /A14 -> /A10
- ARDUINO1 pad A15: /A15 -> /A8
- ARDUINO1 pad A2: /A2 -> /A3
- ARDUINO1 pad A3: /A3 -> /A1
- ARDUINO1 pad A4: /A4 -> /A6
- ARDUINO1 pad A5: /A5 -> /A4
- ARDUINO1 pad A6: /A6 -> /A2
- ARDUINO1 pad A7: /A7 -> /A0
- ARDUINO1 pad A8: /A8 -> /A15
- ARDUINO1 pad A9: /A9 -> /A13
- U1 pad 3: /LED_PWR -> /LIGHTS
Routing:
- net /IO4: track 18.0 -> 93.2 mm
- net /IO7: track 17.1 -> 86.8 mm
- net /BNC_A: track 105.8 -> 36.3 mm, vias 1 -> 0
- net /IO6: track 18.1 -> 84.9 mm
- net /ENC_A: track 51.8 -> 117.2 mm, vias 1 -> 2
- net /IO5: track 20.6 -> 79.0 mm, vias 0 -> 2
- net /IO2: track 20.5 -> 76.3 mm
- net /IO31: track 109.9 -> 56.0 mm, vias 0 -> 2
- net /IO0: track 23.5 -> 73.2 mm
- net /IO1: track 29.3 -> 75.7 mm, vias 0 -> 2
- net /LED_PWR: track 43.1 -> 3.61 mm, vias 1 -> 0
- net /IO3: track 45.4 -> 78.0 mm
- net /IO15: track 74.3 -> 45.5 mm, vias 0 -> 2
- net /A8: track 48.4 -> 76.1 mm, vias 2 -> 1
- net /A13: track 86.6 -> 60.5 mm
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- added copper zone on B.Cu, net GND
- added copper zone on F.Cu, net VAA
- removed copper zone on B.Cu, net VAA
Other:
- board text added: "2.1x5.5 Center +"
- board text added: "A0-7"
- board text added: "A8-15"
- board text added: "IO0-7"
- board text added: "IO16-23"
- board text added: "IO24-31"
- board text added: "IO8-15"
- board text added: "Janelia Modular Device mixed_signal_controller model_number: 1120 08/2015 version 1.2"
- board text added: "https://github.com/janelia-modular-devices"
- board text removed: "12V_DC_DC"
- board text removed: "Janelia Modular Device mixed_signal_controller model_number: 1120 05/2015 version 1.1"
- board text removed: "https://github.com/janelia-modular-devices/modular-devices"
