File: pcb/mixed_signal_controller.sch (KiCad schematic (older format))
At the start: 64 parts, among them P1 PWR_JACK_2.5x5.5, P2 HEADER_01X03, P3 BNC_DOUBLE_RA, P4 HEADER_02X08_SMD, P5 HEADER_02X08_SMD, P6 HEADER_02X08_SMD, P7 HEADER_02X08_SMD, SW1 SPST_SERIES_M, SW2 KT_SWITCH, U1 MAX6817, U2 MAX6817, U3 TLE723X, U4 TLE723X, U5 TLE723X, U6 TLE723X

Commit message: Finished pcb v1.0.
Parts:
- removed C6, C7, C8, C9: 0.1uF, mixed_signal_controller:SM1210, symbol 0.1uF
- removed D10, D11, D12, D13, D14, D15, D16, D17, D18, D19, D2, D20, D21, D22, D23, D24, D25, D26, D27, D28, D29, D3, D30, D31, D32, D33, D4, D5, D6, D7, D8, D9: LED_24V, mixed_signal_controller:LED_555-3XXX, symbol LED_24V
- removed P4, P5, P6, P7: HEADER_02X08_SMD, mixed_signal_controller:HEADER_02x08_SMD, symbol HEADER_02X08_SMD
- removed U3, U4, U5, U6: TLE723X, mixed_signal_controller:TLE723X, symbol TLE723X
- added P4: HEADER_02X05_SMD, mixed_signal_controller:HEADER_02x05_SMD, symbol HEADER_02X05_SMD
Connections:
- net IN is gone; now on net BNC_A: ARDUINO1.48 (D48/ICP5/PL1)
- net +5V: now also P4.1 (P1)
- net BNC_A: no longer ARDUINO1.A0 (A0/PF0)
- net GND: now also P4.2 (P2)
- net A1: now reaches ARDUINO1.A1 (A1/PF1)
- net A1: now also P4.4 (P4)
- net A2: now reaches ARDUINO1.A2 (A2/PF2)
- net A2: now also P4.5 (P5)
- net A3: now reaches ARDUINO1.A3 (A3/PF3)
- net A3: now also P4.6 (P6)
- net A4: now reaches ARDUINO1.A4 (A4/TCK/PF4)
- net A4: now also P4.7 (P7)
- net A5: now reaches ARDUINO1.A5 (A5/TMS/PF5)
- net A5: now also P4.8 (P8)
- net A6: now reaches ARDUINO1.A6 (A6/TDO/PF6)
- net A6: now also P4.9 (P9)
- net A7: now reaches ARDUINO1.A7 (A7/TDI/PF7)
- net A7: now also P4.10 (P10)
- net CS: no longer names the net of ARDUINO1.49 (D49/ICP4/PL0)
- net MISO: no longer names the net of ARDUINO1.50 (D50/MISO/PCINT3/PB3)
- net MOSI: no longer names the net of ARDUINO1.51 (D51/MOSI/PCINT2/PB2)
- net RST: no longer names the net of ARDUINO1.RST
- net SCK: no longer names the net of ARDUINO1.52 (D52/SCK/PCINT1/PB1)
- new net A0: ARDUINO1.A0 (A0/PF0), P4.3 (P3)
- no-connect marks 65 -> 63

Commit message: Finished pcb v1.1.
Parts:
- removed P1: PWR_JACK_2.5x5.5, mixed_signal_controller:DCJACK_2PIN_HIGHCURRENT, symbol PWR_JACK_2.5x5.5
- removed REG1: CONV_DC_DC_12V_1A, mixed_signal_controller:DC_DC_CONV_R78C, symbol CONV_DC_DC_12V_1A
- added P1: PWR_JACK_2.1x5.5, mixed_signal_controller:DCJACK_2PIN_HIGHCURRENT, symbol PWR_JACK_2.1x5.5
- added P5: HEADER_02X05_SMD, mixed_signal_controller:HEADER_02x05_SMD, symbol HEADER_02X05_SMD
- added P6, P7, P8, P9: HEADER_02X07_SMD, mixed_signal_controller:HEADER_02x07_SMD, symbol HEADER_02X07_SMD
Connections:
- net V_IN is gone; now on net VAA: ARDUINO1.V_IN, C2.1
- net +5V: now also P5.1 (P1), P6.5 (P5), P7.5 (P5), P8.5 (P5), P9.5 (P5)
- net GND: now also P1.2 (P2), P5.2 (P2), P6.2 (P2), P6.4 (P4), P6.6 (P6), P7.2 (P2), P7.4 (P4), P7.6 (P6), P8.2 (P2), P8.4 (P4), P8.6 (P6), P9.2 (P2), P9.4 (P4), P9.6 (P6)
- net VAA: now also P1.1 (P1), P6.1 (P1), P6.3 (P3), P7.1 (P1), P7.3 (P3), P8.1 (P1), P8.3 (P3), P9.1 (P1), P9.3 (P3)
- net IO4: now reaches ARDUINO1.10 (D10/PWM/OC2A/PCINT4/PB4)
- net IO4: now also P6.11 (P11)
- net IO5: now reaches ARDUINO1.11 (D11/PWM/OC1A/PCINT5/PB5)
- net IO5: now also P6.12 (P12)
- net IO6: now reaches ARDUINO1.12 (D12/PWM/OC1B/PCINT6/PB6)
- net IO6: now also P6.13 (P13)
- net IO7: now reaches ARDUINO1.13 (D13/PWM/OC0A/OC1C/PCINT7/PB7)
- net IO7: now also P6.14 (P14)
- net IO8: now reaches ARDUINO1.22 (D22/AD0/PA0)
- net IO8: now also P7.7 (P7)
- net IO9: now reaches ARDUINO1.23 (D23/AD1/PA1)
- net IO9: now also P7.8 (P8)
- net IO10: now reaches ARDUINO1.24 (D24/AD2/PA2)
- net IO10: now also P7.9 (P9)
- net IO11: now reaches ARDUINO1.25 (D25/AD3/PA3)
- net IO11: now also P7.10 (P10)
- net IO12: now reaches ARDUINO1.26 (D26/AD4/PA4)
- net IO12: now also P7.11 (P11)
- net IO13: now reaches ARDUINO1.27 (D27/AD5/PA5)
- net IO13: now also P7.12 (P12)
- net IO14: now reaches ARDUINO1.28 (D28/AD6/PA6)
- net IO14: now also P7.13 (P13)
- net IO15: now reaches ARDUINO1.29 (D29/AD7/PA7)
- net IO15: now also P7.14 (P14)
- net IO16: now reaches ARDUINO1.30 (D30/A15/PC7)
- net IO16: now also P8.7 (P7)
- net IO17: now reaches ARDUINO1.31 (D31/A14/PC6)
- net IO17: now also P8.8 (P8)
- net IO18: now reaches ARDUINO1.32 (D32/A13/PC5)
- net IO18: now also P8.9 (P9)
- net IO19: now reaches ARDUINO1.33 (D33/A12/PC4)
- net IO19: now also P8.10 (P10)
- net IO20: now reaches ARDUINO1.34 (D34/A11/PC3)
- net IO20: now also P8.11 (P11)
- net IO21: now reaches ARDUINO1.35 (D35/A10/PC2)
- net IO21: now also P8.12 (P12)
- net IO22: now reaches ARDUINO1.36 (D36/A9/PC1)
- net IO22: now also P8.13 (P13)
- net IO23: now reaches ARDUINO1.37 (D37/A8/PC0)
- net IO23: now also P8.14 (P14)
- net IO31: now reaches ARDUINO1.38 (D38/T0/PD7)
- net IO31: now also P9.14 (P14)
- net IO30: now reaches ARDUINO1.39 (D39/ALE/PG2)
- net IO30: now also P9.13 (P13)
- net IO29: now reaches ARDUINO1.40 (D40/RD/PG1)
- net IO29: now also P9.12 (P12)
- net IO28: now reaches ARDUINO1.41 (D41/WR/PG0)
- net IO28: now also P9.11 (P11)
- net IO27: now reaches ARDUINO1.42 (D42/PL7)
- net IO27: now also P9.10 (P10)
- net IO26: now reaches ARDUINO1.43 (D43/PL6)
- net IO26: now also P9.9 (P9)
- net IO25: now reaches ARDUINO1.44 (D44/PWM/OC5C/PL5)
- net IO25: now also P9.8 (P8)
- net IO24: now reaches ARDUINO1.45 (D45/PWM/OC5B/PL4)
- net IO24: now also P9.7 (P7)
- net IO0: now reaches ARDUINO1.6 (D6/PWM/OC4A/PH3)
- net IO0: now also P6.7 (P7)
- net IO1: now reaches ARDUINO1.7 (D7/PWM/OC4B/PH4)
- net IO1: now also P6.8 (P8)
- net IO2: now reaches ARDUINO1.8 (D8/PWM/OC4C/PH5)
- net IO2: now also P6.9 (P9)
- net IO3: now reaches ARDUINO1.9 (D9/PWM/OC2B/PH6)
- net IO3: now also P6.10 (P10)
- net A10: now reaches ARDUINO1.A10 (A10/PCINT18/PK2)
- net A10: now also P5.5 (P5)
- net A11: now reaches ARDUINO1.A11 (A11/PCINT19/PK3)
- net A11: now also P5.6 (P6)
- net A12: now reaches ARDUINO1.A12 (A12/PCINT20/PK4)
- net A12: now also P5.7 (P7)
- net A13: now reaches ARDUINO1.A13 (A13/PCINT21/PK5)
- net A13: now also P5.8 (P8)
- net A14: now reaches ARDUINO1.A14 (A14/PCINT22/PK6)
- net A14: now also P5.9 (P9)
- net A15: now reaches ARDUINO1.A15 (A15/PCINT23/PK7)
- net A15: now also P5.10 (P10)
- net A8: now reaches ARDUINO1.A8 (A8/PCINT16/PK0)
- net A8: now also P5.3 (P3)
- net A9: now reaches ARDUINO1.A9 (A9/PCINT17/PK1)
- net A9: now also P5.4 (P4)
- no-connect marks 63 -> 23
Other:
- moved on the sheet: C1, C2, D1, P4, R3, SW1

Commit message: SPST switch -> DPST switch.
Parts:
- removed R3: 5.11k, mixed_signal_controller:SM1210, symbol 5.11k
- removed SW1: SPST_SERIES_M, mixed_signal_controller:SPST_SERIES_M, symbol SPST_SERIES_M
- added SW1: DPST_SERIES_M, mixed_signal_controller:DPST_SERIES_M, symbol DPST_SERIES_M
Connections:
- net A0: now also ARDUINO1.A7 (A7/TDI/PF7); no longer ARDUINO1.A0 (A0/PF0)
- net A1: now also ARDUINO1.A3 (A3/PF3); no longer ARDUINO1.A1 (A1/PF1)
- net A10: now also ARDUINO1.A14 (A14/PCINT22/PK6); no longer ARDUINO1.A10 (A10/PCINT18/PK2)
- net A11: now also ARDUINO1.A10 (A10/PCINT18/PK2); no longer ARDUINO1.A11 (A11/PCINT19/PK3)
- net A12: now also ARDUINO1.A13 (A13/PCINT21/PK5); no longer ARDUINO1.A12 (A12/PCINT20/PK4)
- net A13: now also ARDUINO1.A9 (A9/PCINT17/PK1); no longer ARDUINO1.A13 (A13/PCINT21/PK5)
- net A14: now also ARDUINO1.A12 (A12/PCINT20/PK4); no longer ARDUINO1.A14 (A14/PCINT22/PK6)
- net A15: now also ARDUINO1.A8 (A8/PCINT16/PK0); no longer ARDUINO1.A15 (A15/PCINT23/PK7)
- net A2: now also ARDUINO1.A6 (A6/TDO/PF6); no longer ARDUINO1.A2 (A2/PF2)
- net A3: now also ARDUINO1.A2 (A2/PF2); no longer ARDUINO1.A3 (A3/PF3)
- net A4: now also ARDUINO1.A5 (A5/TMS/PF5); no longer ARDUINO1.A4 (A4/TCK/PF4)
- net A5: now also ARDUINO1.A1 (A1/PF1); no longer ARDUINO1.A5 (A5/TMS/PF5)
- net A6: now also ARDUINO1.A4 (A4/TCK/PF4); no longer ARDUINO1.A6 (A6/TDO/PF6)
- net A7: now also ARDUINO1.A0 (A0/PF0); no longer ARDUINO1.A7 (A7/TDI/PF7)
- net A8: now also ARDUINO1.A15 (A15/PCINT23/PK7); no longer ARDUINO1.A8 (A8/PCINT16/PK0)
- net A9: now also ARDUINO1.A11 (A11/PCINT19/PK3); no longer ARDUINO1.A9 (A9/PCINT17/PK1)
- net BNC_A: now also ARDUINO1.12 (D12/PWM/OC1B/PCINT6/PB6); no longer ARDUINO1.48 (D48/ICP5/PL1)
- net GND: now also SW1.6
- net IO0: now also ARDUINO1.29 (D29/AD7/PA7); no longer ARDUINO1.6 (D6/PWM/OC4A/PH3)
- net IO1: now also ARDUINO1.28 (D28/AD6/PA6); no longer ARDUINO1.7 (D7/PWM/OC4B/PH4)
- net IO10: now also ARDUINO1.35 (D35/A10/PC2); no longer ARDUINO1.24 (D24/AD2/PA2)
- net IO11: now also ARDUINO1.34 (D34/A11/PC3); no longer ARDUINO1.25 (D25/AD3/PA3)
- net IO12: now also ARDUINO1.33 (D33/A12/PC4); no longer ARDUINO1.26 (D26/AD4/PA4)
- net IO13: now also ARDUINO1.32 (D32/A13/PC5); no longer ARDUINO1.27 (D27/AD5/PA5)
- net IO14: now also ARDUINO1.31 (D31/A14/PC6); no longer ARDUINO1.28 (D28/AD6/PA6)
- net IO15: now also ARDUINO1.30 (D30/A15/PC7); no longer ARDUINO1.29 (D29/AD7/PA7)
- net IO16: now also ARDUINO1.45 (D45/PWM/OC5B/PL4); no longer ARDUINO1.30 (D30/A15/PC7)
- net IO17: now also ARDUINO1.44 (D44/PWM/OC5C/PL5); no longer ARDUINO1.31 (D31/A14/PC6)
- net IO18: now also ARDUINO1.43 (D43/PL6); no longer ARDUINO1.32 (D32/A13/PC5)
- net IO19: now also ARDUINO1.42 (D42/PL7); no longer ARDUINO1.33 (D33/A12/PC4)
- net IO2: now also ARDUINO1.27 (D27/AD5/PA5); no longer ARDUINO1.8 (D8/PWM/OC4C/PH5)
- net IO20: now also ARDUINO1.41 (D41/WR/PG0); no longer ARDUINO1.34 (D34/A11/PC3)
- net IO21: now also ARDUINO1.40 (D40/RD/PG1); no longer ARDUINO1.35 (D35/A10/PC2)
- net IO22: now also ARDUINO1.39 (D39/ALE/PG2); no longer ARDUINO1.36 (D36/A9/PC1)
- net IO23: now also ARDUINO1.38 (D38/T0/PD7); no longer ARDUINO1.37 (D37/A8/PC0)
- net IO24: now also ARDUINO1.53 (D53/SS/PCINT0/PB0); no longer ARDUINO1.45 (D45/PWM/OC5B/PL4)
- net IO25: now also ARDUINO1.52 (D52/SCK/PCINT1/PB1); no longer ARDUINO1.44 (D44/PWM/OC5C/PL5)
- net IO26: now also ARDUINO1.51 (D51/MOSI/PCINT2/PB2); no longer ARDUINO1.43 (D43/PL6)
- net IO27: now also ARDUINO1.50 (D50/MISO/PCINT3/PB3); no longer ARDUINO1.42 (D42/PL7)
- net IO28: now also ARDUINO1.49 (D49/ICP4/PL0); no longer ARDUINO1.41 (D41/WR/PG0)
- net IO29: now also ARDUINO1.48 (D48/ICP5/PL1); no longer ARDUINO1.40 (D40/RD/PG1)
- net IO3: now also ARDUINO1.26 (D26/AD4/PA4); no longer ARDUINO1.9 (D9/PWM/OC2B/PH6)
- net IO30: now also ARDUINO1.47 (D47/T5/PL2); no longer ARDUINO1.39 (D39/ALE/PG2)
- net IO31: now also ARDUINO1.46 (D46/PWM/OC5A/PL3); no longer ARDUINO1.38 (D38/T0/PD7)
- net IO4: now also ARDUINO1.25 (D25/AD3/PA3); no longer ARDUINO1.10 (D10/PWM/OC2A/PCINT4/PB4)
- net IO5: now also ARDUINO1.24 (D24/AD2/PA2); no longer ARDUINO1.11 (D11/PWM/OC1A/PCINT5/PB5)
- net IO6: now also ARDUINO1.23 (D23/AD1/PA1); no longer ARDUINO1.12 (D12/PWM/OC1B/PCINT6/PB6)
- net IO7: now also ARDUINO1.22 (D22/AD0/PA0); no longer ARDUINO1.13 (D13/PWM/OC0A/OC1C/PCINT7/PB7)
- net IO8: now also ARDUINO1.37 (D37/A8/PC0); no longer ARDUINO1.22 (D22/AD0/PA0)
- net IO9: now also ARDUINO1.36 (D36/A9/PC1); no longer ARDUINO1.23 (D23/AD1/PA1)
- net LED_PWR: now also SW1.3; no longer U1.3 (IN2)
- net VAA: now also SW1.2
- net D_LED_PWR renamed D_LIGHTS
- new net LIGHTS: SW1.5, U1.3 (IN2)
Other:
- moved on the sheet: D1, P4, P5, P6, P7, P8, P9
